File: Board/micromouse/micromouse.kicad_pcb (KiCad board)
At the start: 2 copper layers, 50 x 53 mm, 91 parts, among them J1 Conn_01x02_Pin, J2 Conn_02x03_Odd_Even, J3 Conn_01x06_Pin, J4 Conn_01x06_Pin, J5 Conn_01x06_Pin, J6 Conn_01x06_Pin, M1 Motor_DC, M2 Motor_DC, Q1 DMN63D8L-7, Q10 DMN63D8L-7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

Commit message: レビュー対応
Parts:
- added G***: LOGO, LOGO, B.Cu at (151.1, 100.0)
- C14, C15, C16, C17, C18, C19, C8: value C -> 0.1u
- C2, C3: value C -> 1u
- C4, C5, C6, C7: value 0.01u -> 0.1u
- D10, D11, D12, D13: footprint LED_SMD:LED_0603_1608Metric -> LED_SMD:LED_0402_1005Metric
- J1: footprint Connector_JST:JST_PH_B2B-PH-SM4-TB_1x02-1MP_P2.00mm_Vertical -> Connector_JST:JST_PH_B2B-PH-K_1x02_P2.00mm_Vertical
- R13, R17, R5, R9: value R -> 10
- R21: value R -> 6.8k
- R22: value R -> 15k
- R24, R25, R26, R27: value R -> 1k
- R28: value R -> 10k
- moved SW4 2.18 mm to (118.5, 118.2), turned to 180 degrees
- moved R33 2.05 mm to (118.1, 116.3)
- moved J1 1.33 mm to (119.5, 84.4)
- moved Q7 0.60 mm to (122.8, 91.3)
- moved C1 0.58 mm to (123.4, 94.8)
- moved R32 0.30 mm to (156.7, 90.1)
- moved J4 0.10 mm to (140.0, 103.9)
- moved J5 0.10 mm to (140.0, 96.1)
Connections:
- Q7 pad 1: GND -> Net-(Q7-G)
- R1 pad 2: unconnected-(R1-Pad2) -> +3.3V
- R2 pad 2: unconnected-(R2-Pad2) -> +3.3V
- R23 pad 1: unconnected-(R23-Pad1) -> GND
- R3 pad 2: Net-(SW1-A) -> Net-(Q7-G)
- R33 pad 1: /NRST -> +3.3V
- R33 pad 2: GND -> /NRST
- SW1 pad 1: Net-(SW1-A) -> Net-(Q7-G)
- SW4 pad 1: /NRST -> GND
- SW4 pad 2: +3.3V -> /NRST
Routing:
- net +3.3V: track 232.9 -> 253.6 mm, vias 8 -> 9
- net Net-(Q7-G): track 0.00 -> 8.91 mm
- net Net-(SW1-A): track 4.37 -> 0.00 mm
- net Net-(J1-Pin_1): track 2.60 -> 0.00 mm
- net Net-(D7-K): track 8.03 -> 6.54 mm
- net GND: vias 174 -> 166
