File: Board/micromouse/ENC.kicad_sch (KiCad schematic)
At the start: 2 parts, among them J3 Conn_01x06_Pin, U5 MAQ473GQE-AEC1-Z

Commit message: 部品型番、URLを追加
Parts:
- J3: manf# (none) -> -
Changed lines of the file:
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@@
+      (effects (font (size 1.27 1.27)) hide)
+    )
+    (property "manf#" "-" (at 109.22 96.52 0)
       (effects (font (size 1.27 1.27)) hide)
     )
